File: 01_Hardware/REV_B.kicad_pcb (KiCad board)
At the start: 2 copper layers, 65 x 30 mm, 87 parts, among them J1 RaspberryPi, J10 Conn_01x03, J11 Conn_01x03, J12 Conn_01x03, J13 Conn_01x08, J14 Conn_01x01, J2 Conn_01x02, J3 Conn_01x02, J4 Conn_01x02, J5 Conn_01x08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

Commit message: Fix missing GND connection to PushButton
Connections:
- SW1 pad 2: Net-(SW1-Pad2) -> GND
Routing:
- net Net-(SW1-Pad2): track 6.50 -> 0.00 mm
Changed lines of the file:
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@@
-(kicad_pcb (version 20171130) (host pcbnew 6.0.0-rc1-unknown-829ba27~65~ubuntu17.10.1)
+(kicad_pcb (version 20171130) (host pcbnew 5.0.2-bee76a0~70~ubuntu18.04.1)
   (general
     (thickness 1.6)
     (drawings 109)
-    (tracks 928)
+    (tracks 927)
     (zones 0)
     (modules 87)
-    (nets 82)
+    (nets 81)
   )
   (page A4)
@@
     (zone_45_only no)
     (trace_min 0.1524)
+    (segment_width 0.1)
+    (edge_width 0.15)
     (via_size 0.6858)
     (via_drill 0.3302)
@@
     (uvia_min_size 0.2)
     (uvia_min_drill 0.1)
-    (edge_width 0.15)
-    (segment_width 0.1)
     (pcb_text_width 0.3)
     (pcb_text_size 1.5 1.5)
@@
     (pad_drill 1)
     (pad_to_mask_clearance 0.0508)
+    (solder_mask_min_width 0.25)
     (aux_axis_origin 0 0)
     (visible_elements FEFDFF7F)
@@
   (net 79 "Net-(R19-Pad1)")
   (net 80 "Net-(R20-Pad1)")
-  (net 81 "Net-(SW1-Pad2)")
   (net_class Default "This is the default net class."
     (clearance 0.1524)
@@
     (add_net "Net-(R48-Pad2)")
     (add_net "Net-(R9-Pad2)")
-    (add_net "Net-(SW1-Pad2)")
     (add_net PUSH_BUTTON)
     (add_net SPI0_CLK_LV)
@@
     (fp_circle (center 3.25 2.25) (end 1.25 2.5) (layer F.Fab) (width 0.1))
     (pad 2 thru_hole circle (at 0 4.5 90) (size 2 2) (drill 1.1) (layers *.Cu *.Mask)
-      (net 81 "Net-(SW1-Pad2)"))
+      (net 4 GND))
     (pad 1 thru_hole circle (at 0 0 90) (size 2 2) (drill 1.1) (layers *.Cu *.Mask)
       (net 75 "Net-(R48-Pad2)"))
     (pad 2 thru_hole circle (at 6.5 4.5 90) (size 2 2) (drill 1.1) (layers *.Cu *.Mask)
-      (net 81 "Net-(SW1-Pad2)"))
+      (net 4 GND))
     (pad 1 thru_hole circle (at 6.5 0 90) (size 2 2) (drill 1.1) (layers *.Cu *.Mask)
       (net 75 "Net-(R48-Pad2)"))
@@
   (segment (start 55.1366 13.0683) (end 57.1881 13.0683) (width 0.9144) (layer F.Cu) (net 4))
   (segment (start 57.2516 9.1313) (end 53.3781 9.1313) (width 0.9144) (layer F.Cu) (net 4))
-  (via (at 51.2572 27.2796) (size 0.6858) (drill 0.3302) (layers F.Cu B.Cu) (net 4))
   (segment (start 24.13 9.13) (end 25.908 9.13) (width 0.4064) (layer B.Cu) (net 5) (status 30))
   (segment (start 25.908 9.13) (end 27.94 9.13) (width 0.4064) (layer B.Cu) (net 5) (status 30))
@@
   (via (at 56.388 25.8064) (size 0.6858) (drill 0.3302) (layers F.Cu B.Cu) (net 80))
   (segment (start 41.7484 21.7344) (end 52.316 21.7344) (width 0.4064) (layer B.Cu) (net 80))
-  (segment (start 52.6288 28.5284) (end 59.1288 28.5284) (width 0.4064) (layer B.Cu) (net 81) (status 30))
+  (via (at 51.2572 27.2796) (size 0.6858) (drill 0.3302) (layers F.Cu B.Cu) (net 4))
   (zone (net 4) (net_name GND) (layer F.Cu) (hatch edge 0.508)
     (connect_pads (clearance 0.1524))
